Commit message: add kinova, stablebaselines agent

File: urdf/kinova_robotiq_85.urdf (robot description, URDF)
Before this commit: robot robotiq_arg2f_85_model, 12 links, 11 joints
Links:
- removed link prismatic_x_link
- added link base_link, mass 1.697; collision mesh filename=../meshes/kinova/base_link.STL; visual mesh filename=../meshes/kinova/base_link.STL
- added link bracelet_link, mass 0.5; collision mesh filename=../meshes/kinova/bracelet_with_vision_link.STL; visual mesh filename=../meshes/kinova/bracelet_with_vision_link.STL
- added link camera_color_frame
- added link camera_depth_frame
- added link camera_link
- added link end_effector_link
- added link forearm_link, mass 0.9302; collision mesh filename=../meshes/kinova/forearm_link.STL; visual mesh filename=../meshes/kinova/forearm_link.STL
- added link half_arm_1_link, mass 1.1636; collision mesh filename=../meshes/kinova/half_arm_1_link.STL; visual mesh filename=../meshes/kinova/half_arm_1_link.STL
- added link half_arm_2_link, mass 1.1636; collision mesh filename=../meshes/kinova/half_arm_2_link.STL; visual mesh filename=../meshes/kinova/half_arm_2_link.STL
- added link shoulder_link, mass 1.3773; collision mesh filename=../meshes/kinova/shoulder_link.STL; visual mesh filename=../meshes/kinova/shoulder_link.STL
- added link spherical_wrist_1_link, mass 0.6781; collision mesh filename=../meshes/kinova/spherical_wrist_1_link.STL; visual mesh filename=../meshes/kinova/spherical_wrist_1_link.STL
- added link spherical_wrist_2_link, mass 0.6781; collision mesh filename=../meshes/kinova/spherical_wrist_2_link.STL; visual mesh filename=../meshes/kinova/spherical_wrist_2_link.STL
- added link tool_frame
- added link world
Joints:
- removed joint prismatic_x_joint
- added joint camera_module: type fixed, parent end_effector_link, child camera_link, origin xyz=0 0.05639 -0.00305 rpy=3.14159265358979 3.14159265358979 0
- added joint color_module: type fixed, parent end_effector_link, child camera_color_frame, origin xyz=0 0.05639 -0.00305 rpy=3.14159265358979 3.14159265358979 0
- added joint depth_module: type fixed, parent end_effector_link, child camera_depth_frame, origin xyz=0.0275 0.066 -0.00305 rpy=3.14159265358979 3.14159265358979 0
- added joint end_effector: type fixed, parent bracelet_link, child end_effector_link, origin xyz=0 0 -0.0615250000000001 rpy=3.14159265358979 1.09937075168372E-32 0, axis 0 0 0
- added joint joint_1: type continuous, parent base_link, child shoulder_link, origin xyz=0 0 0.15643 rpy=3.1416 2.7629E-18 -4.9305E-36, axis 0 0 1, limit effort=39 velocity=1.3963
- added joint joint_2: type revolute, parent shoulder_link, child half_arm_1_link, origin xyz=0 0.005375 -0.12838 rpy=1.5708 2.1343E-17 -1.1102E-16, axis 0 0 1, limit lower=-2.41 upper=2.41 effort=39 velocity=1.3963
- added joint joint_3: type continuous, parent half_arm_1_link, child half_arm_2_link, origin xyz=0 -0.21038 -0.006375 rpy=-1.5708 1.2326E-32 -2.9122E-16, axis 0 0 1, limit effort=39 velocity=1.3963
- added joint joint_4: type revolute, parent half_arm_2_link, child forearm_link, origin xyz=0 0.006375 -0.21038 rpy=1.5708 -6.6954E-17 -1.6653E-16, axis 0 0 1, limit lower=-2.66 upper=2.66 effort=39 velocity=1.3963
- added joint joint_5: type continuous, parent forearm_link, child spherical_wrist_1_link, origin xyz=0 -0.20843 -0.006375 rpy=-1.5708 2.2204E-16 -6.373E-17, axis 0 0 1, limit effort=9 velocity=1.2218
- added joint joint_6: type revolute, parent spherical_wrist_1_link, child spherical_wrist_2_link, origin xyz=0 0.00017505 -0.10593 rpy=1.5708 9.2076E-28 -8.2157E-15, axis 0 0 1, limit lower=-2.23 upper=2.23 effort=9 velocity=1.2218
- added joint joint_7: type continuous, parent spherical_wrist_2_link, child bracelet_link, origin xyz=0 -0.10593 -0.00017505 rpy=-1.5708 -5.5511E-17 9.6396E-17, axis 0 0 1, limit effort=9 velocity=1.2218
- added joint robotiq_85_base_joint: type fixed, parent end_effector_link, child robotiq_arg2f_base_link, origin xyz=0 0 0 rpy=0 0 0
- added joint tool_frame_joint: type fixed, parent end_effector_link, child tool_frame, origin xyz=0 0 0 rpy=0 0 0, axis 0 0 0
- added joint world_arm_joint: type fixed, parent world, child base_link, origin xyz=0 0 0 rpy=0.0 0.0 0
